Commit message: added robot model and sensors

File: src/robot_urdf/urdf/robot.urdf.xacro (robot description, xacro)
@@ -21,4 +21,7 @@
   <xacro:property name="wheelRadius" value="0.0762" />
   <xacro:property name="wheelOffset" value="0.25" />
+  <xacro:property name="camMass" value="0.05" />
+  <xacro:property name="camWidth" value="0.1016" />
+  <xacro:property name="camRadius" value="0.0127" />
   <link name="base_link">
     <visual>
@@ -138,3 +141,54 @@
     <origin xyz="${-wheelOffset} ${baseWidth /2} 0"/>
   </joint>
+  <!-- Sensors -->
+  <link name="t265_pose_frame">
+    <visual>
+      <geometry>
+        <cylinder length="${camWidth}" radius="${camRadius}"/>
+      </geometry>
+      <origin rpy="0 1.57075 1.57075" xyz="0 0 0"/>
+      <material name="white"/>
+    </visual>
+    <collision>
+      <geometry>
+        <cylinder length="${camWidth}" radius="${camRadius}"/>
+      </geometry>
+      <origin rpy="0 1.57075 1.57075" xyz="0 0 0"/>
+    </collision>
+    <inertial>
+      <mass value="${camMass}"/>
+      <inertia ixx="0.4" ixy="0.0" ixz="0.0" iyy="0.4" iyz="0.0" izz="0.2"/>
+    </inertial>
+  </link>
+  <joint name="base_to_t265_pose_frame" type="fixed">
+    <parent link="base_link"/>
+    <child link="t265_pose_frame"/>
+    <axis xyz="0 1 0"/>
+    <origin xyz="0.25 0 .2"/>
+  </joint>
+  <link name="d435_link">
+    <visual>
+      <geometry>
+        <cylinder length="${camWidth}" radius="${camRadius}"/>
+      </geometry>
+      <origin rpy="0 1.57075 1.57075" xyz="0 0 0"/>
+      <material name="white"/>
+    </visual>
+    <collision>
+      <geometry>
+        <cylinder length="${camWidth}" radius="${camRadius}"/>
+      </geometry>
+      <origin rpy="0 1.57075 1.57075" xyz="0 0 0"/>
+    </collision>
+    <inertial>
+      <mass value="${camMass}"/>
+      <inertia ixx="0.4" ixy="0.0" ixz="0.0" iyy="0.4" iyz="0.0" izz="0.2"/>
+    </inertial>
+  </link>
+  <joint name="base_to_d435_link" type="fixed">
+    <parent link="base_link"/>
+    <child link="d435_link"/>
+    <axis xyz="0 1 0"/>
+    <origin xyz="0.25 0 0.2508"/>
+  </joint>
 </robot>

Commit message: updated

File: src/robot_urdf/urdf/robot.urdf.xacro (robot description, xacro)
@@ -192,3 +192,28 @@
     <origin xyz="0.25 0 0.2508"/>
   </joint>
+  <link name="laser">
+    <visual>
+      <geometry>
+        <cylinder length="${camWidth}" radius="${camRadius}"/>
+      </geometry>
+      <origin rpy="0 1.57075 1.57075" xyz="0 0 0"/>
+      <material name="white"/>
+    </visual>
+    <collision>
+      <geometry>
+        <cylinder length="${camWidth}" radius="${camRadius}"/>
+      </geometry>
+      <origin rpy="0 1.57075 1.57075" xyz="0 0 0"/>
+    </collision>
+    <inertial>
+      <mass value="${camMass}"/>
+      <inertia ixx="0.4" ixy="0.0" ixz="0.0" iyy="0.4" iyz="0.0" izz="0.2"/>
+    </inertial>
+  </link>
+  <joint name="base_to_laser" type="fixed">
+    <parent link="base_link"/>
+    <child link="laser"/>
+    <axis xyz="0 1 0"/>
+    <origin xyz="0.25 0 0.2508"/>
+  </joint>
 </robot>

Commit message: updated

File: src/robot_urdf/urdf/robot.urdf.xacro (robot description, xacro)
@@ -215,5 +215,5 @@
     <child link="laser"/>
     <axis xyz="0 1 0"/>
-    <origin xyz="0.25 0 0.2508"/>
+    <origin xyz="0.25 0 0.2508" rpy="0 0 3.1415"/>
   </joint>
 </robot>

Commit message: updated urdf

File: src/robot_urdf/urdf/robot.urdf.xacro (robot description, xacro)
@@ -13,6 +13,6 @@
     <color rgba="0 1 0 0.5"/>
   </material>
-  <xacro:property name="baseLength" value="0.8" />
-  <xacro:property name="baseWidth" value="0.6" />
+  <xacro:property name="baseLength" value="0.8255" />
+  <xacro:property name="baseWidth" value="0.6985" />
   <xacro:property name="baseHeight" value="0.1" />
   <xacro:property name="baseMass" value="27" />
@@ -165,5 +165,5 @@
     <child link="t265_pose_frame"/>
     <axis xyz="0 1 0"/>
-    <origin xyz="0.25 0 .2"/>
+    <origin xyz="0.2159 0 .2"/>
   </joint>
   <link name="d435_link">
@@ -190,5 +190,5 @@
     <child link="d435_link"/>
     <axis xyz="0 1 0"/>
-    <origin xyz="0.25 0 0.2508"/>
+    <origin xyz="0.2159 0 0.2508"/>
   </joint>
   <link name="laser">
@@ -215,5 +215,5 @@
     <child link="laser"/>
     <axis xyz="0 1 0"/>
-    <origin xyz="0.25 0 0.2508" rpy="0 0 3.1415"/>
+    <origin xyz="0.2159 0 0.2508" rpy="0 0 3.1415"/>
   </joint>
 </robot>

Commit message: updated

File: src/robot_urdf/urdf/robot.urdf.xacro (robot description, xacro)
@@ -165,5 +165,5 @@
     <child link="t265_pose_frame"/>
     <axis xyz="0 1 0"/>
-    <origin xyz="0.2159 0 .2"/>
+    <origin xyz="-0.1524 0 .2"/>
   </joint>
   <link name="d435_link">
@@ -190,5 +190,5 @@
     <child link="d435_link"/>
     <axis xyz="0 1 0"/>
-    <origin xyz="0.2159 0 0.2508"/>
+    <origin xyz="-0.1524 0 0.2508"/>
   </joint>
   <link name="laser">
@@ -215,5 +215,5 @@
     <child link="laser"/>
     <axis xyz="0 1 0"/>
-    <origin xyz="0.2159 0 0.2508" rpy="0 0 3.1415"/>
+    <origin xyz="-0.1524 0 0.2508" rpy="0 0 3.1415"/>
   </joint>
 </robot>

Commit message: Added between frame for realsense

File: src/robot_urdf/urdf/robot.urdf.xacro (robot description, xacro)
@@ -142,4 +142,29 @@
   </joint>
   <!-- Sensors -->
+  <link name="t265_odom_frame">
+    <visual>
+      <geometry>
+        <cylinder length="${camWidth}" radius="${camRadius}"/>
+      </geometry>
+      <origin rpy="0 1.57075 1.57075" xyz="0 0 0"/>
+      <material name="white"/>
+    </visual>
+    <collision>
+      <geometry>
+        <cylinder length="${camWidth}" radius="${camRadius}"/>
+      </geometry>
+      <origin rpy="0 1.57075 1.57075" xyz="0 0 0"/>
+    </collision>
+    <inertial>
+      <mass value="${camMass}"/>
+      <inertia ixx="0.4" ixy="0.0" ixz="0.0" iyy="0.4" iyz="0.0" izz="0.2"/>
+    </inertial>
+  </link>
+  <joint name="base_to_t265_odom_frame" type="fixed">
+    <parent link="base_link"/>
+    <child link="t265_odom_frame"/>
+    <axis xyz="0 1 0"/>
+    <origin xyz="0.1524 0 .2"/>
+  </joint>
   <link name="t265_pose_frame">
     <visual>
@@ -162,8 +187,8 @@
   </link>
   <joint name="base_to_t265_pose_frame" type="fixed">
-    <parent link="base_link"/>
+    <parent link="t265_odom_frame"/>
     <child link="t265_pose_frame"/>
     <axis xyz="0 1 0"/>
-    <origin xyz="-0.1524 0 .2"/>
+    <origin xyz="0 0 0"/>
   </joint>
   <link name="d435_link">
@@ -190,5 +215,5 @@
     <child link="d435_link"/>
     <axis xyz="0 1 0"/>
-    <origin xyz="-0.1524 0 0.2508"/>
+    <origin xyz="0.1524 0 0.2508"/>
   </joint>
   <link name="laser">
@@ -215,5 +240,5 @@
     <child link="laser"/>
     <axis xyz="0 1 0"/>
-    <origin xyz="-0.1524 0 0.2508" rpy="0 0 3.1415"/>
+    <origin xyz="0.127 0 0.2508" rpy="0 0 3.1415"/>
   </joint>
 </robot>

Commit message: updated tf frames

File: src/robot_urdf/urdf/robot.urdf.xacro (robot description, xacro)
@@ -142,5 +142,5 @@
   </joint>
   <!-- Sensors -->
-  <link name="t265_odom_frame">
+  <link name="t265_pose_frame">
     <visual>
       <geometry>
@@ -161,11 +161,11 @@
     </inertial>
   </link>
-  <joint name="base_to_t265_odom_frame" type="fixed">
-    <parent link="base_link"/>
-    <child link="t265_odom_frame"/>
-    <axis xyz="0 1 0"/>
-    <origin xyz="0.1524 0 .2"/>
-  </joint>
-  <link name="t265_pose_frame">
+  <joint name="base_to_t265_pose_frame" type="fixed">
+    <parent link="t265_pose_frame"/>
+    <child link="base_link"/>
+    <axis xyz="0 1 0"/>
+    <origin xyz="-0.1524 0 -0.2"/>
+  </joint>
+  <link name="d435_link">
     <visual>
       <geometry>
@@ -186,11 +186,11 @@
     </inertial>
   </link>
-  <joint name="base_to_t265_pose_frame" type="fixed">
-    <parent link="t265_odom_frame"/>
-    <child link="t265_pose_frame"/>
-    <axis xyz="0 1 0"/>
-    <origin xyz="0 0 0"/>
-  </joint>
-  <link name="d435_link">
+  <joint name="base_to_d435_link" type="fixed">
+    <parent link="base_link"/>
+    <child link="d435_link"/>
+    <axis xyz="0 1 0"/>
+    <origin xyz="0.1524 0 0.2508"/>
+  </joint>
+  <link name="laser">
     <visual>
       <geometry>
@@ -211,29 +211,4 @@
     </inertial>
   </link>
-  <joint name="base_to_d435_link" type="fixed">
-    <parent link="base_link"/>
-    <child link="d435_link"/>
-    <axis xyz="0 1 0"/>
-    <origin xyz="0.1524 0 0.2508"/>
-  </joint>
-  <link name="laser">
-    <visual>
-      <geometry>
-        <cylinder length="${camWidth}" radius="${camRadius}"/>
-      </geometry>
-      <origin rpy="0 1.57075 1.57075" xyz="0 0 0"/>
-      <material name="white"/>
-    </visual>
-    <collision>
-      <geometry>
-        <cylinder length="${camWidth}" radius="${camRadius}"/>
-      </geometry>
-      <origin rpy="0 1.57075 1.57075" xyz="0 0 0"/>
-    </collision>
-    <inertial>
-      <mass value="${camMass}"/>
-      <inertia ixx="0.4" ixy="0.0" ixz="0.0" iyy="0.4" iyz="0.0" izz="0.2"/>
-    </inertial>
-  </link>
   <joint name="base_to_laser" type="fixed">
     <parent link="base_link"/>

Commit message: updated urdf for new robot

File: src/robot_urdf/urdf/robot.urdf.xacro (robot description, xacro)
@@ -13,7 +13,7 @@
     <color rgba="0 1 0 0.5"/>
   </material>
-  <xacro:property name="baseLength" value="0.8255" />
-  <xacro:property name="baseWidth" value="0.6985" />
-  <xacro:property name="baseHeight" value="0.1" />
+  <xacro:property name="baseLength" value="0.8636" />
+  <xacro:property name="baseWidth" value="0.9652" />
+  <xacro:property name="baseHeight" value="0.6096" />
   <xacro:property name="baseMass" value="27" />
   <xacro:property name="wheelMass" value="0.453592" />
@@ -30,4 +30,5 @@
       </geometry>
       <material name="blue"/>
+      <origin rpy="0 0 0" xyz="0 0 0.3"/>
     </visual>
     <collision>
@@ -35,4 +36,5 @@
         <box size="${baseLength} ${baseWidth} ${baseHeight}"/>
       </geometry>
+      <origin rpy="0 0 0" xyz="0 0 0.3"/>
     </collision>
     <inertial>
@@ -165,5 +167,5 @@
     <child link="base_link"/>
     <axis xyz="0 1 0"/>
-    <origin xyz="-0.1524 0 -0.2"/>
+    <origin xyz="-0.381 0 -0.5842"/>
   </joint>
   <link name="d435_link">
@@ -190,5 +192,5 @@
     <child link="d435_link"/>
     <axis xyz="0 1 0"/>
-    <origin xyz="0.1524 0 0.2508"/>
+    <origin xyz="0.381 0 0.6223"/>
   </joint>
   <link name="laser">
@@ -215,5 +217,5 @@
     <child link="laser"/>
     <axis xyz="0 1 0"/>
-    <origin xyz="0.127 0 0.2508" rpy="0 0 3.1415"/>
+    <origin xyz="0.381 0 0.66" rpy="0 0 3.1415"/>
   </joint>
 </robot>
